File: Printer-HAT.kicad_sch (KiCad schematic)
At the start: 38 parts, among them J1 Screw_Terminal, J4 Conn_01x03_Male, K1 SRD-05VDC-SL-C, K2 SLA-05VDC-SL-C, P1 Conn_02x20_Odd_Even, Q2 S8050, Q3 S8050, Q4 Q_Dual_PNP_PNP_C1B1B2C2E2E1, Q5 DMG2305UX-7, U1 LM2596S-5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

Commit message: update screw terminal to 5mm pitch
Parts:
- J1: footprint TerminalBlock:TerminalBlock_bornier-6_P5.08mm -> TerminalBlock_MetzConnect:TerminalBlock_MetzConnect_Type011_RT05506HBWC_1x06_P5.00mm_Horizontal
Changed lines of the file:
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@@
     (property "Reference" "J1" (id 0) (at 191.77 125.5735 0))
     (property "Value" "Screw_Terminal" (id 1) (at 191.77 128.3486 0))
-    (property "Footprint" "TerminalBlock:TerminalBlock_bornier-6_P5.08mm" (id 2) (at 191.77 138.43 0)
+    (property "Footprint" "TerminalBlock_MetzConnect:TerminalBlock_MetzConnect_Type011_RT05506HBWC_1x06_P5.00mm_Horizontal" (id 2) (at 191.77 138.43 0)
       (effects (font (size 1.27 1.27)) hide)
     )
@@
     )
     (path "/dca84cac-ad35-4240-bdbf-f7734aa71de3"
-      (reference "J1") (unit 1) (value "Screw_Terminal") (footprint "TerminalBlock:TerminalBlock_bornier-6_P5.08mm")
+      (reference "J1") (unit 1) (value "Screw_Terminal") (footprint "TerminalBlock_MetzConnect:TerminalBlock_MetzConnect_Type011_RT05506HBWC_1x06_P5.00mm_Horizontal")
     )
     (path "/e2bc1001-dc48-409a-a60c-28e01d5d4087"
