File: pcb/Printer-HAT.kicad_sch (KiCad schematic)
At the start: 38 parts, among them J1 Screw_Terminal, J4 Conn_01x03_Male, K1 SRD-05VDC-SL-C, K2 SLA-05VDC-SL-C, P1 Conn_02x20_Odd_Even, Q2 S8050, Q3 S8050, Q4 Q_Dual_PNP_PNP_C1B1B2C2E2E1, Q5 DMG2305UX-7, U1 LM2596S-5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

Commit message: fix issues with initial pcb
Parts:
- removed Q2, Q3: S8050, Package_TO_SOT_SMD:SOT-23, symbol Transistor_BJT:S8050
- added Q1, Q2: S8050, Package_TO_SOT_SMD:SOT-23, symbol Device:Q_NPN_BEC
- R3: value 3K -> 1K; LCSC C4211 -> C21190; Manufacturer_Part_Number 0603WAF3001T5E -> 0603WAF1001T5E
Connections:
- net +5V: now also R3.2, R4.2
- net +5VD: now also U1.4 (FB); no longer R3.1
- net AUX_PWR: now also K1.5; no longer K1.4
- net GND: now also Q1.2 (E), Q2.2 (E); no longer R4.2
- net GPIO14(TXD0): now also J4.1 (Pin_1)
- net GPIO17(GEN0): now also U2.2; no longer D5.1 (K)
- net GPIO27(GEN2): now also U3.2; no longer D6.1 (K)
- net GPIO4(GCLK): no longer J4.1 (Pin_1)
- net at D7.2 (A), K2.5: now also D5.1 (K), Q1.3 (C)
- net at R10.2: now also Q1.1 (B)
- net at R11.2: now also Q2.1 (B)
- net at D8.2 (A), K1.3: now also D6.1 (K), Q2.3 (C)
- net at D6.2 (A): now also R4.1; no longer U3.2
- net at D5.2 (A): now also R3.1; no longer U2.2
Other:
- moved on the sheet: D5, D6, D7, D8, R6, R7, R8, R9

Commit message: Documentation
Parts:
- J1: LCSC C192771 -> C424695; Manufacturer_Name Ningbo Kangnex Elec -> DIBO; Manufacturer_Part_Number WJ128V-5.0-6P -> DB128V-5.0-3P-BK-S
Changed lines of the file:
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@@
       (effects (font (size 1.27 1.27)) hide)
     )
-    (property "LCSC" "C192771" (id 4) (at 191.77 138.43 0)
+    (property "LCSC" "C424695" (id 4) (at 191.77 138.43 0)
       (effects (font (size 1.27 1.27)) hide)
     )
-    (property "Manufacturer_Name" "Ningbo Kangnex Elec" (id 5) (at 191.77 138.43 0)
+    (property "Manufacturer_Name" "DIBO" (id 5) (at 191.77 138.43 0)
       (effects (font (size 1.27 1.27)) hide)
     )
-    (property "Manufacturer_Part_Number" "WJ128V-5.0-6P" (id 6) (at 191.77 138.43 0)
+    (property "Manufacturer_Part_Number" "DB128V-5.0-3P-BK-S" (id 6) (at 191.77 138.43 0)
       (effects (font (size 1.27 1.27)) hide)
     )
